Commit message: update xbot model and ISCAS museum

File: xbot_description/urdf/robot.xacro (robot description, xacro)
@@ -6,9 +6,10 @@
   name="sick_tim">
   <xacro:include filename="$(find xbot_description)/urdf/sick_tim.urdf.xacro" />
-  <xacro:sick_tim571 name="laser" ros_topic="scan"   />
+  <!-- Choose your laser -->
+  <!--<xacro:sick_tim571 name="laser" ros_topic="scan"   />-->
+  <xacro:rplidarA2 name="laser" ros_topic="scan"   />
   <xacro:include filename="$(find xbot_description)/urdf/materials.xacro" />
-  <xacro:include filename="$(find xbot_description)/urdf/xbot.urdf.xacro" />
-  <xacro:include filename="$(find xbot_description)/urdf/xbot.gazebo" />
-  <xacro:xbot_base/>
-  <!--xacro:include filename="$(find xbot_description)/urdf/sick_tim.gazebo.xacro" /-->
+  <xacro:include filename="$(find xbot_description)/urdf/xbot-u.urdf.xacro" />
+  <xacro:include filename="$(find xbot_description)/urdf/xbot-u.gazebo" />
+  <xacro:xbot2_base/>
 </robot>

File: xbot_description/urdf/sick_tim.urdf.xacro (robot description, xacro)
@@ -4,4 +4,10 @@
   xmlns:sensor="http://playerstage.sourceforge.net/gazebo/xmlschema/#sensor"
   xmlns:xacro="http://ros.org/wiki/xacro">
+  <xacro:macro name="rplidarA2" params="name ros_topic">
+    <xacro:sick_tim name="${name}" ros_topic="${ros_topic}"
+      length="0.06" width="0.06" height="0.079" mass="0.150" z_offset="0.05595"
+      min_range="0.2" max_range="8.0"
+      mesh="package://xbot_description/models/meshes/rplidar.dae" />
+  </xacro:macro>
   <xacro:macro name="sick_tim310" params="name ros_topic">
     <xacro:sick_tim name="${name}" ros_topic="${ros_topic}"
@@ -58,5 +64,6 @@
     <gazebo reference="${link}">
       <material value="Gazebo/LightWood" />
-      <sensor type="ray" name="${name}">
+      <sensor type="gpu_ray" name="${name}">
+      <!--sensor type="ray" name="${name}"-->
         <always_on>true</always_on>
         <update_rate>${update_rate}</update_rate>
@@ -78,5 +85,6 @@
           </range>
         </ray>
-        <plugin name="gazebo_ros_${name}_controller" filename="libgazebo_ros_laser.so">
+        <plugin name="gazebo_ros_${name}_controller" filename="libgazebo_ros_gpu_laser.so">
+        <!-- plugin name="gazebo_ros_${name}_controller" filename="libgazebo_ros_laser.so" -->
           <gaussianNoise>0.01</gaussianNoise>
           <alwaysOn>true</alwaysOn>
