Commit message: delete links above of camera_link

File: xbot_description/urdf/xbot-u.urdf.xacro (robot description, xacro)
@@ -210,15 +210,4 @@
     <child link="camera_link"/>
   </joint>
-  <!-- generate an optical frame http://www.ros.org/reps/rep-0103.html#suffix-frames
-      so that ros and opencv can operate on the camera frame correctly -->
-  <joint name="camera_optical_joint" type="fixed">
-    <!-- these values have to be these values otherwise the gazebo camera image
-        won't be aligned properly with the frame it is supposedly originating from -->
-    <origin xyz="0 0 0" rpy="-1.5708 0 -1.5708"/>
-    <parent link="camera_link"/>
-    <child link="camera_link_optical"/>
-  </joint>
-  <link name="camera_link_optical">
-  </link>
   </xacro:macro>
 </robot>
