Commit message: Release XBot 核心功能 V52 版本
主要变更：
1. 大幅度改进和完善了代码。
2. 添加了机器人启动后播报等功能。
3. 添加了Deb包构建的脚本及配置，为后续进入ROS官方源准备。
4. 其它 bugfix 及 doc 更新。

File: xbot_description/urdf/sick_tim.urdf.xacro (robot description, xacro)
@@ -6,6 +6,6 @@
   <xacro:macro name="rplidarA2" params="name ros_topic">
     <xacro:sick_tim name="${name}" ros_topic="${ros_topic}"
-      length="0.06" width="0.06" height="0.079" mass="0.150" z_offset="0.05595"
-      min_range="0.2" max_range="8.0"
+      length="0.06" width="0.06" height="0.079" mass="0.150" z_offset="0.0308"
+      min_range="0.2" max_range="12.0"
       mesh="package://xbot_description/models/meshes/rplidar.dae" />
   </xacro:macro>
@@ -33,5 +33,5 @@
       <parent link="${name}_mount_link" />
       <child link="${name}" />
-      <origin rpy="0 0 0" xyz="0 0 ${z_offset}"/>
+      <origin rpy="0 0 3.1415926" xyz="0 0 ${z_offset}"/>
     </joint>
     <link name="${name}">

File: xbot_description/urdf/xbot-u.urdf.xacro (robot description, xacro)
@@ -4,5 +4,5 @@
   xmlns:sensor="http://playerstage.sourceforge.net/gazebo/xmlschema/#sensor"
   xmlns:xacro="http://ros.org/wiki/xacro">
-  <xacro:macro name="xbot2_base">
+  <xacro:macro name="xbot_base">
   <link name="base_footprint"/>
   <joint name="base_footprint_to_base" type="fixed">
@@ -66,5 +66,5 @@
     <parent link="base_link"/>
     <child link="laser_mount_link"/>
-    <origin rpy="0 0 0" xyz=".114 0 .17"/>
+    <origin rpy="0 0 0" xyz=".120 0 .205"/>
   </joint>
   <link name="imu_link"/>
@@ -73,5 +73,5 @@
     <parent link="base_link"/>
     <child link="imu_link"/>
-    <origin rpy="0 0 0" xyz="0 0 .2"/>
+    <origin rpy="0 0 0" xyz="0.0454 -0.0157 1.1724"/>
   </joint>
   <link name="left_wheel">
@@ -152,5 +152,5 @@
     <parent link="base_link"/>
     <child link="yaw_platform"/>
-    <origin rpy="0 0 0" xyz="0 0 1.305"/>
+    <origin rpy="0 0 0" xyz="0 0 1.232"/>
     <limit effort="100" velocity="100" lower="-1.57" upper="1.57" />
     <dynamics damping="0.0" friction="10.0"/>
@@ -179,5 +179,5 @@
     <parent link="yaw_platform"/>
     <child link="pitch_platform"/>
-    <origin rpy="0 0 0" xyz="0 0 0"/>
+    <origin rpy="0 0 0" xyz="0.0208 0 0.01325"/>
     <limit effort="100" velocity="100" lower="-1.57" upper="1.57" />
     <dynamics damping="0.0" friction="10.0"/>
